Commit message: Commit

File: kuka_agilus_support/urdf/kr4_r600.urdf.xacro (robot description, xacro)
@@ -32,5 +32,5 @@
   <link name="world"/>
   <!-- robot links, joints -->
-  <xacro:kuka_kr4_r600_robot prefix="$(arg prefix)" package_name="kuka_agilus_support"/>
+  <xacro:kuka_kr4_r600_robot prefix="$(arg prefix)" package_name="kuka_agilus_support" base_collision="${False}"/>
   <!-- default world - base_link joint -->
   <joint name="$(arg prefix)world-base_link" type="fixed">

File: kuka_agilus_support/urdf/kr4_r600_macro.xacro (robot description, xacro)
@@ -1,13 +1,15 @@
 <?xml version="1.0" encoding="UTF-8"?>
 <robot xmlns:xacro="http://www.ros.org/wiki/xacro" name="kr4_r600">
-  <xacro:macro name="kuka_kr4_r600_robot" params="prefix package_name">
+  <xacro:macro name="kuka_kr4_r600_robot" params="prefix package_name base_collision:=true">
     <link name="${prefix}base"/>
     <link name="${prefix}base_link">
-      <collision>
-        <geometry>
-          <mesh filename="package://${package_name}/meshes/kr4_r600/collision/base_link.stl"/>
-        </geometry>
-        <origin rpy="0.0 -0.0 0.0" xyz="0.0 0.0 0.0"/>
-      </collision>
+      <xacro:if value="${base_collision}">
+        <collision>
+          <geometry>
+            <mesh filename="package://${package_name}/meshes/kr4_r600/collision/base_link.stl"/>
+          </geometry>
+          <origin rpy="0.0 -0.0 0.0" xyz="0.0 0.0 0.0"/>
+        </collision>
+      </xacro:if>
       <inertial>
         <inertia ixx="0.01774610228117179" ixy="0.0" ixz="0.0" iyy="0.028906995427589975" iyz="0.0" izz="0.029332705372297367"/>

File: kuka_kr_moveit_config/srdf/kr_arm.srdf.xacro (robot description, xacro)
@@ -6,5 +6,12 @@
 <robot xmlns:xacro="http://www.ros.org/wiki/xacro" name="$(arg robot_name)">
   <xacro:arg name="prefix" default=""/>
+  <xacro:property name="robot_name_value" value="$(arg robot_name)"/>
   <xacro:include filename="kr_arm_macro.xacro"/>
   <xacro:kuka_kr_arm prefix="$(arg prefix)"/>
+  <xacro:if value="${robot_name_value == 'kr4_r600'}">
+    <disable_collisions link1="ashpick_cell_table" link2="zed_camera_center" reason="Never"/>
+    <disable_collisions link1="ashpick_wall_left" link2="zed_camera_center" reason="Never"/>
+    <disable_collisions link1="ashpick_wall_right" link2="zed_camera_center" reason="Never"/>
+    <disable_collisions link1="ashpick_wall_back" link2="zed_camera_center" reason="Never"/>
+  </xacro:if>
 </robot>
